File: relay_dip_v01.brd (EAGLE design)
At the start: 50 x 50 mm, 47 parts, among them IC2 DS2432P

Commit message: t
Parts:
- removed SV1: (no value), con-lstb:MA04-1
- added R11: 10k, rcl:R0805
- added S1: SWITCH-MOMENTARY-2SMD, SparkFun-Electromechanical:TACTILE-SWITCH-SMD
- added SV2: (no value), con-lstb:MA06-1
- moved U$5 26.2 mm to (21.3, 48.0), turned to 270 degrees
- moved U$4 8.81 mm to (40.5, 24.4), turned to 0 degrees
- moved U$10 7.70 mm to (38.1, 31.8), turned to 0 degrees
- moved C1 1.00 mm to (28.3, 44.5)
- moved C2 1.00 mm to (37.4, 44.5)
- moved C4 1.00 mm to (19.0, 44.5)
- moved C5 1.00 mm to (10.0, 44.5)
- renumbered EARTH to E.
Connections:
- new net N$1: R11.2, S1.1, SV2.5
- new net N$6: R11.1, SV2.6
- net GND: now also S1.3
- net P0: now also SV2.4; no longer SV1.4
- net P2: now also SV2.3; no longer SV1.3
- net P4: now also SV2.2; no longer SV1.2
- net P6: now also SV2.1; no longer SV1.1
Routing:
- net N$1: track 0.00 -> 10.4 mm
- net GND: track 11.6 -> 20.2 mm
- net N$6: track 0.00 -> 6.79 mm
- net VCC: track 184.4 -> 185.5 mm
- net EARTH: track 59.8 -> 60.6 mm
- net P6: track 28.1 -> 28.6 mm
Other:
- board text added: "JKW v0.1"
- board text added: "RELAY DIP I"
- board text removed: "CHIP bat connector"
- board text removed: "Input 5V Close left"
- board text removed: "JKW v0.32"
- board text removed: "ONION DIP IIb"
