File: relay_dip_v01.sch (EAGLE design)
At the start: 47 parts, among them IC2 DS2432P

Commit message: t
Parts:
- removed SV1: (no value), con-lstb:MA04-1
- added R11: 10k, rcl:R-EU_R0805
- added S1: SWITCH-MOMENTARY-2SMD, SparkFun-Electromechanical:SWITCH-MOMENTARY-2SMD
- added SV2: (no value), con-lstb:MA06-1
- renumbered EARTH to E.
Connections:
- new net N$1: R11.2, S1.1, SV2.5
- new net N$6: R11.1, SV2.6
- net GND: now also S1.2
- net P0: now also SV2.4; no longer SV1.4
- net P2: now also SV2.3; no longer SV1.3
- net P4: now also SV2.2; no longer SV1.2
- net P6: now also SV2.1; no longer SV1.1
Changed lines of the file:
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@@
 <layer number="56" name="wert" color="7" fill="1" visible="no" active="no"/>
 <layer number="57" name="tCAD" color="7" fill="1" visible="no" active="no"/>
+<layer number="59" name="tCarbon" color="7" fill="1" visible="no" active="no"/>
+<layer number="60" name="bCarbon" color="7" fill="1" visible="no" active="no"/>
 <layer number="90" name="Modules" color="5" fill="1" visible="yes" active="yes"/>
 <layer number="91" name="Nets" color="2" fill="1" visible="yes" active="yes"/>
@@
 <layer number="115" name="antenne" color="9" fill="1" visible="no" active="no"/>
 <layer number="116" name="Patch_BOT" color="9" fill="4" visible="yes" active="yes"/>
+<layer number="118" name="Rect_Pads" color="7" fill="1" visible="yes" active="yes"/>
 <layer number="121" name="_tsilk" color="7" fill="1" visible="yes" active="yes"/>
 <layer number="122" name="_bsilk" color="7" fill="1" visible="yes" active="yes"/>
@@
 <layer number="127" name="_tValues" color="7" fill="1" visible="yes" active="yes"/>
 <layer number="128" name="_bValues" color="7" fill="1" visible="yes" active="yes"/>
+<layer number="129" name="Mask" color="7" fill="1" visible="yes" active="yes"/>
 <layer number="131" name="tAdjust" color="7" fill="1" visible="yes" active="yes"/>
 <layer number="132" name="bAdjust" color="7" fill="1" visible="yes" active="yes"/>
@@
 <layer number="223" name="223bmp" color="24" fill="1" visible="no" active="no"/>
 <layer number="224" name="224bmp" color="25" fill="1" visible="no" active="no"/>
+<layer number="225" name="225bmp" color="7" fill="1" visible="yes" active="yes"/>
+<layer number="226" name="226bmp" color="7" fill="1" visible="yes" active="yes"/>
+<layer number="227" name="227bmp" color="7" fill="1" visible="yes" active="yes"/>
+<layer number="228" name="228bmp" color="7" fill="1" visible="yes" active="yes"/>
+<layer number="229" name="229bmp" color="7" fill="1" visible="yes" active="yes"/>
+<layer number="230" name="230bmp" color="7" fill="1" visible="yes" active="yes"/>
+<layer number="231" name="231bmp" color="7" fill="1" visible="yes" active="yes"/>
 <layer number="248" name="Housing" color="7" fill="1" visible="yes" active="yes"/>
 <layer number="249" name="Edge" color="7" fill="1" visible="yes" active="yes"/>
@@
 <layer number="251" name="SMDround" color="12" fill="11" visible="no" active="no"/>
 <layer number="254" name="cooling" color="7" fill="1" visible="yes" active="yes"/>
+<layer number="255" name="routoute" color="7" fill="1" visible="yes" active="yes"/>
 </layers>
 <schematic xreflabel="%F%N/%S.%C%R" xrefpart="/%S.%C%R">
@@
 <part name="GND4" library="supply1" deviceset="GND" device=""/>
 <part name="P+1" library="supply1" deviceset="VCC" device=""/>
-<part name="EARTH" library="wirepad" deviceset="WIREPAD" device="3,17/1,3"/>
+<part name="E." library="wirepad" deviceset="WIREPAD" device="3,17/1,3"/>
 <part name="N4" library="wirepad" deviceset="WIREPAD" device="3,17/1,3"/>
 <part name="IC2" library="1wire" deviceset="DS2432" device="P"/>
@@
 <part name="C4" library="rcl" deviceset="CPOL-US" device="150CLZ-0810"/>
 <part name="C5" library="rcl" deviceset="CPOL-US" device="150CLZ-0810"/>
-<part name="SV1" library="con-lstb" deviceset="MA04-1" device=""/>
 <part name="SV3" library="con-lstb" deviceset="MA03-2" device=""/>
 <part name="JP1" library="adafruit" deviceset="PINHD-1X3" device=""/>
@@
 <part name="C2" library="rcl" deviceset="CPOL-US" device="150CLZ-0810"/>
 <part name="GND7" library="supply1" deviceset="GND" device=""/>
+<part name="S1" library="SparkFun-Electromechanical" deviceset="SWITCH-MOMENTARY-2" device="SMD"/>
+<part name="R11" library="rcl" deviceset="R-EU_" device="R0805" value="10k"/>
+<part name="SV2" library="con-lstb" deviceset="MA06-1" device=""/>
 </parts>
 <sheets>
@@
 <instance part="GND4" gate="1" x="114.3" y="548.64"/>
 <instance part="P+1" gate="VCC" x="167.64" y="574.04" rot="MR0"/>
-<instance part="EARTH" gate="G$1" x="218.44" y="571.5" rot="MR0"/>
+<instance part="E." gate="G$1" x="218.44" y="571.5" rot="MR0"/>
 <instance part="N4" gate="G$1" x="210.82" y="556.26" rot="MR0"/>
 <instance part="IC2" gate="G$1" x="15.24" y="462.28"/>
@@
 <instance part="C4" gate="G$1" x="45.72" y="368.3"/>
 <instance part="C5" gate="G$1" x="53.34" y="368.3"/>
-<instance part="SV1" gate="1" x="246.38" y="515.62"/>
 <instance part="SV3" gate="1" x="317.5" y="520.7"/>
 <instance part="JP1" gate="A" x="-15.24" y="454.66" rot="R180"/>
@@
 <instance part="C2" gate="G$1" x="88.9" y="386.08"/>
 <instance part="GND7" gate="1" x="88.9" y="375.92" rot="MR0"/>
+<instance part="S1" gate="G$1" x="299.72" y="500.38"/>
+<instance part="R11" gate="G$1" x="284.48" y="508" rot="R270"/>
+<instance part="SV2" gate="1" x="246.38" y="518.16"/>
 </instances>
 <busses>
@@
 <wire x1="88.9" y1="378.46" x2="88.9" y2="381" width="0.1524" layer="91"/>
 </segment>
+<segment>
+<pinref part="S1" gate="G$1" pin="2"/>
+<wire x1="304.8" y1="500.38" x2="317.5" y2="500.38" width="0.1524" layer="91"/>
+<label x="309.88" y="500.38" size="1.778" layer="95"/>
+</segment>
 </net>
 <net name="P0" class="0">
@@
 </segment>
 <segment>
-<pinref part="SV1" gate="1" pin="4"/>
 <wire x1="254" y1="518.16" x2="266.7" y2="518.16" width="0.1524" layer="91"/>
+<label x="259.08" y="518.16" size="1.778" layer="95"/>
+<pinref part="SV2" gate="1" pin="4"/>
 </segment>
 </net>
@@
 </segment>
 <segment>
-<pinref part="EARTH" gate="G$1" pin="P"/>
+<pinref part="E." gate="G$1" pin="P"/>
 <wire x1="215.9" y1="571.5" x2="203.2" y2="571.5" width="0.1524" layer="91"/>
 <label x="203.2" y="571.5" size="1.778" layer="95"/>
@@
 </segment>
 <segment>
-<pinref part="SV1" gate="1" pin="3"/>
 <wire x1="254" y1="515.62" x2="266.7" y2="515.62" width="0.1524" layer="91"/>
+<label x="259.08" y="515.62" size="1.778" layer="95"/>
+<pinref part="SV2" gate="1" pin="3"/>
 </segment>
 </net>
@@
 </segment>
 <segment>
-<pinref part="SV1" gate="1" pin="2"/>
 <wire x1="254" y1="513.08" x2="266.7" y2="513.08" width="0.1524" layer="91"/>
+<label x="259.08" y="513.08" size="1.778" layer="95"/>
+<pinref part="SV2" gate="1" pin="2"/>
 </segment>
 </net>
@@
 </segment>
 <segment>
-<pinref part="SV1" gate="1" pin="1"/>
 <wire x1="254" y1="510.54" x2="266.7" y2="510.54" width="0.1524" layer="91"/>
-</segment>
-</net>
+<label x="259.08" y="510.54" size="1.778" layer="95"/>
+<pinref part="SV2" gate="1" pin="1"/>
+</segment>
+</net>
+<net name="N$1" class="0">
+<segment>
+<pinref part="SV2" gate="1" pin="5"/>
+<wire x1="254" y1="520.7" x2="276.86" y2="520.7" width="0.1524" layer="91"/>
+<wire x1="276.86" y1="520.7" x2="276.86" y2="500.38" width="0.1524" layer="91"/>
+<pinref part="S1" gate="G$1" pin="1"/>
+<wire x1="276.86" y1="500.38" x2="284.48" y2="500.38" width="0.1524" layer="91"/>
+<pinref part="R11" gate="G$1" pin="2"/>
+<wire x1="284.48" y1="500.38" x2="294.64" y2="500.38" width="0.1524" layer="91"/>
+<wire x1="284.48" y1="502.92" x2="284.48" y2="500.38" width="0.1524" layer="91"/>
+<junction x="284.48" y="500.38"/>
+</segment>
+</net>
+<net name="N$6" class="0">
+<segment>
+<pinref part="SV2" gate="1" pin="6"/>
+<wire x1="254" y1="523.24" x2="284.48" y2="523.24" width="0.1524" layer="91"/>
+<pinref part="R11" gate="G$1" pin="1"/>
+<wire x1="284.48" y1="523.24" x2="284.48" y2="513.08" width="0.1524" layer="91"/>
+</segment>
+</net>
