File: schematics/v1_ordered/relay_dip_v011.brd (EAGLE design)
At the start: 50 x 50 mm, 51 parts, among them IC1 74HCT04D, IC2 DS2432P

Commit message: v2
Parts:
- moved U$10 17.9 mm to (34.6, 49.4), turned to 270 degrees
- moved S1 14.9 mm to (45.4, 43.6), turned to 90 degrees
- moved E 14.5 mm to (46.2, 33.0)
- moved P 14.5 mm to (46.2, 28.0)
- moved B1 8.92 mm to (44.7, 43.5), turned to 180 degrees
- moved C2 4.90 mm to (28.6, 44.5)
- moved C4 2.45 mm to (19.6, 44.5)
- moved C5 0.75 mm to (10.8, 44.5)
Routing:
- net N$5: track 43.2 -> 76.0 mm
- net GND: track 58.2 -> 33.7 mm, vias 16 -> 17
- net EARTH: track 59.0 -> 39.3 mm
- net VCC: track 169.8 -> 160.6 mm
- net N$1: track 20.4 -> 29.2 mm
- net P6: track 66.0 -> 63.1 mm
- net N$11: track 53.6 -> 51.0 mm
- net 3V: track 77.6 -> 75.7 mm
- net P2: track 27.4 -> 28.7 mm
- net N$2: track 38.2 -> 39.0 mm
- net PHASE: track 101.3 -> 100.7 mm
