File: schematics/v1_ordered/relay_dip_v02.brd (EAGLE design)
At the start: 50 x 50 mm, 51 parts, among them IC1 74HCT04D, IC2 DS2432P

Commit message: v2
Parts:
- removed E, P: WIREPAD3,17/1,3, wirepad:3,17/1,3
- added COM_IN, PHASE_IN: WIREPAD3,17/1,3, wirepad:3,17/1,3
- moved U$10 17.9 mm to (34.6, 49.4), turned to 270 degrees
- moved S1 14.9 mm to (45.4, 43.6), turned to 90 degrees
- moved R11 13.9 mm to (40.5, 33.8)
- moved B1 8.92 mm to (44.7, 43.5), turned to 180 degrees
- moved C2 4.90 mm to (28.6, 44.5)
- moved C4 2.45 mm to (19.6, 44.5)
- moved U$5 2.25 mm to (39.8, 4.30)
- moved C5 0.75 mm to (10.8, 44.5)
- renumbered E. to COM_OUT
Connections:
- net EARTH: now also COM_IN.1; no longer E.1
- net PHASE: now also PHASE_IN.1; no longer P.1
Routing:
- net N$5: track 43.2 -> 76.0 mm
- net GND: track 58.2 -> 33.7 mm, vias 16 -> 17
- net EARTH: track 59.0 -> 39.3 mm
- net 3V: track 77.6 -> 62.7 mm
- net VCC: track 169.8 -> 160.6 mm
- net N$1: track 20.4 -> 29.4 mm
- net P6: track 66.0 -> 63.1 mm
- net N$11: track 53.6 -> 51.0 mm
- net P2: track 27.4 -> 28.7 mm
- net N$2: track 38.2 -> 39.0 mm
- net PHASE: track 101.3 -> 100.7 mm
