File: schematics/v1_ordered/relay_dip_v02.sch (EAGLE design)
At the start: 52 parts, among them IC1 74HCT04D, IC2 DS2432P

Commit message: v2
Parts:
- removed C1: EMVE500ADA221MJA0G, rcl:CPOL-US150CLZ-0810
- C2, C4, C5: value (none) -> EMZR500ADA221MHA0G
- renumbered E to COM_IN, E. to COM_OUT, P to PHASE_IN
Connections:
- removed net N$6: R11.1, SV4.8
- new net 3V: IC1P.VCC, R10.1, R11.1, R6.1, R8.1, R9.1, SV4.8
- new net N$11: IC1E.O, U$12.G
- new net N$2: IC1A.O, U$3.G
- new net N$7: IC1B.O, U$7.G
- new net N$9: IC1C.O, U$9.G
- net GND: now also IC1P.GND; no longer C1.-, R10.2, R6.2, R8.2, R9.2
- net N$5: no longer C1.+
- net P0: now also IC1A.I, R8.2; no longer R8.1, U$3.G
- net P2: now also IC1B.I, R6.2; no longer R6.1, U$7.G
- net P4: now also IC1C.I, R9.2; no longer R9.1, U$9.G
- net P6: now also IC1E.I, R10.2; no longer R10.1, U$12.G
Other:
- note added: "220uF 50VDC 800 mA 4x $0,66 EMZR500ADA221MHA0G"
- note added: "512-DF005S 50V 1.5A $0.446"
- note removed: "220uF 50VDC 375 mA 4x $1"
- note removed: "ABS15J RGG 600V 1.5A $0.42"
- moved on the sheet: IC1A, IC1B, IC1C, IC1E, IC1F, R10, R6, R8, R9
